File: hardware/glcd2usb-m8.sch (EAGLE design)
At the start: 19 parts, among them IC1 MEGA8-P, Q1 12MHz, T1 BC547

Commit message: fix connections
Parts:
- added IC2: LM1117-3.3, v-reg:LM317MBSTT3
- R1, R2: value 220 -> 68; device resistor:R-EU_R0603 -> resistor:R-EU_0207/2V
- R3: value 10k -> 1k5; device resistor:R-EU_R0603 -> resistor:R-EU_0207/2V
- R6: device resistor:R-EU_R0603 -> resistor:R-EU_0207/2V
Connections:
- removed net MOSI: JP6.1
- new net +5V: IC2.IN, JP1.19, JP1.2, JP3.4, R4.E
- net GND: now also IC2.ADJ
- net SCK: now also JP6.1
- net VCC: now also IC2.OUT; no longer JP1.19, JP1.2, JP3.4, R4.E
Other:
- moved on the sheet: C1
Changed lines of the file:
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@@
 <part name="IC1" library="atmel" deviceset="MEGA8-P" device=""/>
 <part name="T1" library="transistor" deviceset="BC547" device=""/>
-<part name="R1" library="resistor" deviceset="R-EU_" device="R0603" value="220"/>
-<part name="R2" library="resistor" deviceset="R-EU_" device="R0603" value="220"/>
-<part name="R3" library="resistor" deviceset="R-EU_" device="R0603" value="10k"/>
+<part name="R1" library="resistor" deviceset="R-EU_" device="0207/2V" value="68"/>
+<part name="R2" library="resistor" deviceset="R-EU_" device="0207/2V" value="68"/>
+<part name="R3" library="resistor" deviceset="R-EU_" device="0207/2V" value="1k5"/>
 <part name="C1" library="resistor" deviceset="C-EU" device="C0603"/>
 <part name="R4" library="pot" deviceset="TRIM_EU-" device="B25P"/>
@@
 <part name="GND2" library="supply1" deviceset="GND" device=""/>
 <part name="R5" library="resistor" deviceset="R-EU_" device="0204/2V" value="47"/>
-<part name="R6" library="resistor" deviceset="R-EU_" device="R0603" value="4k7"/>
+<part name="R6" library="resistor" deviceset="R-EU_" device="0207/2V" value="4k7"/>
 <part name="JP3" library="pinhead" deviceset="PINHD-1X4" device="" value="USB"/>
 <part name="P+1" library="supply1" deviceset="VCC" device=""/>
-<part name="P+2" library="supply1" deviceset="VCC" device=""/>
 <part name="GND3" library="supply1" deviceset="GND" device=""/>
-<part name="P+3" library="supply1" deviceset="VCC" device=""/>
 <part name="Q1" library="crystal" deviceset="CRYSTAL" device="HC49S" value="12MHz"/>
 <part name="C2" library="resistor" deviceset="C-EU" device="C0603" value="22"/>
@@
 <part name="JP7" library="pinhead" deviceset="PINHD-1X1" device="" value="MOSI"/>
 <part name="GND6" library="supply1" deviceset="GND" device=""/>
+<part name="IC2" library="v-reg" deviceset="LM317?*" device="MBSTT3" value="LM1117-3.3"/>
+<part name="GND7" library="supply1" deviceset="GND" device=""/>
+<part name="P+5" library="supply1" deviceset="+5V" device=""/>
+<part name="P+3" library="supply1" deviceset="+5V" device=""/>
+<part name="P+2" library="supply1" deviceset="+5V" device=""/>
 </parts>
 <sheets>
@@
 <instance part="R2" gate="G$1" x="-81.28" y="12.7"/>
 <instance part="R3" gate="G$1" x="-73.66" y="25.4" rot="R90"/>
-<instance part="C1" gate="G$1" x="-88.9" y="22.86"/>
+<instance part="C1" gate="G$1" x="-71.12" y="43.18"/>
 <instance part="R4" gate="1" x="63.5" y="15.24"/>
 <instance part="GND1" gate="1" x="-93.98" y="2.54"/>
@@
 <instance part="R6" gate="G$1" x="60.96" y="-45.72"/>
 <instance part="JP3" gate="A" x="-104.14" y="15.24" rot="R180"/>
-<instance part="P+1" gate="VCC" x="-93.98" y="35.56"/>
-<instance part="P+2" gate="VCC" x="66.04" y="-25.4" rot="R90"/>
+<instance part="P+1" gate="VCC" x="-71.12" y="58.42"/>
 <instance part="GND3" gate="1" x="76.2" y="27.94" rot="R180"/>
-<instance part="P+3" gate="VCC" x="71.12" y="27.94"/>
 <instance part="Q1" gate="G$1" x="-38.1" y="7.62" rot="R90"/>
 <instance part="C2" gate="G$1" x="-45.72" y="12.7" rot="R90"/>
@@
 <instance part="JP7" gate="G$1" x="-50.8" y="-20.32"/>
 <instance part="GND6" gate="1" x="-91.44" y="-40.64"/>
+<instance part="IC2" gate="G$1" x="-81.28" y="50.8"/>
+<instance part="GND7" gate="1" x="-81.28" y="33.02"/>
+<instance part="P+5" gate="1" x="-93.98" y="58.42"/>
+<instance part="P+3" gate="1" x="71.12" y="27.94"/>
+<instance part="P+2" gate="1" x="66.04" y="-25.4" rot="R90"/>
 </instances>
 <busses>
@@
 <pinref part="GND1" gate="1" pin="GND"/>
 <pinref part="JP3" gate="A" pin="1"/>
-<pinref part="C1" gate="G$1" pin="2"/>
-<wire x1="-88.9" y1="17.78" x2="-88.9" y2="10.16" width="0.1524" layer="91"/>
-<wire x1="-88.9" y1="10.16" x2="-93.98" y2="10.16" width="0.1524" layer="91"/>
-<junction x="-93.98" y="10.16"/>
 </segment>
 <segment>
@@
 <pinref part="GND6" gate="1" pin="GND"/>
 </segment>
+<segment>
+<pinref part="IC2" gate="G$1" pin="ADJ"/>
+<pinref part="GND7" gate="1" pin="GND"/>
+<wire x1="-81.28" y1="43.18" x2="-81.28" y2="38.1" width="0.1524" layer="91"/>
+<pinref part="C1" gate="G$1" pin="2"/>
+<wire x1="-81.28" y1="38.1" x2="-81.28" y2="35.56" width="0.1524" layer="91"/>
+<wire x1="-71.12" y1="38.1" x2="-81.28" y2="38.1" width="0.1524" layer="91"/>
+<junction x="-81.28" y="38.1"/>
+</segment>
 </net>
 <net name="MD-" class="0">
@@
 </net>
 <net name="VCC" class="0">
-<segment>
-<wire x1="-101.6" y1="17.78" x2="-93.98" y2="17.78" width="0.1524" layer="91"/>
-<wire x1="-93.98" y1="17.78" x2="-93.98" y2="30.48" width="0.1524" layer="91"/>
-<pinref part="R3" gate="G$1" pin="2"/>
-<wire x1="-93.98" y1="30.48" x2="-93.98" y2="33.02" width="0.1524" layer="91"/>
-<wire x1="-93.98" y1="30.48" x2="-88.9" y2="30.48" width="0.1524" layer="91"/>
-<wire x1="-88.9" y1="30.48" x2="-73.66" y2="30.48" width="0.1524" layer="91"/>
-<junction x="-93.98" y="30.48"/>
-<pinref part="JP3" gate="A" pin="4"/>
-<pinref part="P+1" gate="VCC" pin="VCC"/>
-<pinref part="C1" gate="G$1" pin="1"/>
-<wire x1="-88.9" y1="30.48" x2="-88.9" y2="25.4" width="0.1524" layer="91"/>
-<junction x="-88.9" y="30.48"/>
-</segment>
-<segment>
-<wire x1="83.82" y1="17.78" x2="71.12" y2="17.78" width="0.1524" layer="91"/>
-<pinref part="P+3" gate="VCC" pin="VCC"/>
-<wire x1="71.12" y1="17.78" x2="71.12" y2="22.86" width="0.1524" layer="91"/>
-<pinref part="R4" gate="1" pin="E"/>
-<wire x1="71.12" y1="22.86" x2="71.12" y2="25.4" width="0.1524" layer="91"/>
-<wire x1="63.5" y1="20.32" x2="63.5" y2="22.86" width="0.1524" layer="91"/>
-<wire x1="63.5" y1="22.86" x2="71.12" y2="22.86" width="0.1524" layer="91"/>
-<junction x="71.12" y="22.86"/>
-<label x="73.66" y="17.78" size="1.778" layer="95"/>
-<pinref part="JP1" gate="A" pin="2"/>
-</segment>
 <segment>
 <pinref part="IC1" gate="G$1" pin="AVCC"/>
@@
 </segment>
 <segment>
-<pinref part="JP1" gate="A" pin="19"/>
-<pinref part="P+2" gate="VCC" pin="VCC"/>
-<wire x1="83.82" y1="-25.4" x2="68.58" y2="-25.4" width="0.1524" layer="91"/>
+<pinref part="C1" gate="G$1" pin="1"/>
+<pinref part="P+1" gate="VCC" pin="VCC"/>
+<wire x1="-71.12" y1="45.72" x2="-71.12" y2="50.8" width="0.1524" layer="91"/>
+<pinref part="IC2" gate="G$1" pin="OUT"/>
+<wire x1="-71.12" y1="50.8" x2="-71.12" y2="55.88" width="0.1524" layer="91"/>
+<wire x1="-73.66" y1="50.8" x2="-71.12" y2="50.8" width="0.1524" layer="91"/>
+<junction x="-71.12" y="50.8"/>
+<wire x1="-63.5" y1="50.8" x2="-71.12" y2="50.8" width="0.1524" layer="91"/>
+<wire x1="-63.5" y1="50.8" x2="-63.5" y2="33.02" width="0.1524" layer="91"/>
+<pinref part="R3" gate="G$1" pin="2"/>
+<wire x1="-63.5" y1="33.02" x2="-73.66" y2="33.02" width="0.1524" layer="91"/>
+<wire x1="-73.66" y1="33.02" x2="-73.66" y2="30.48" width="0.1524" layer="91"/>
 </segment>
 </net>
@@
 <label x="27.94" y="-30.48" size="1.778" layer="95"/>
 </segment>
-</net>
-<net name="MOSI" class="0">
 <segment>
 <pinref part="JP6" gate="G$1" pin="1"/>
@@
 </segment>
 </net>
+<net name="+5V" class="0">
+<segment>
+<pinref part="JP3" gate="A" pin="4"/>
+<wire x1="-101.6" y1="17.78" x2="-93.98" y2="17.78" width="0.1524" layer="91"/>
+<wire x1="-93.98" y1="17.78" x2="-93.98" y2="50.8" width="0.1524" layer="91"/>
+<pinref part="IC2" gate="G$1" pin="IN"/>
+<pinref part="P+5" gate="1" pin="+5V"/>
+<wire x1="-93.98" y1="50.8" x2="-88.9" y2="50.8" width="0.1524" layer="91"/>
+<wire x1="-93.98" y1="55.88" x2="-93.98" y2="50.8" width="0.1524" layer="91"/>
+<junction x="-93.98" y="50.8"/>
+</segment>
+<segment>
+<wire x1="83.82" y1="17.78" x2="71.12" y2="17.78" width="0.1524" layer="91"/>
+<wire x1="71.12" y1="17.78" x2="71.12" y2="22.86" width="0.1524" layer="91"/>
+<pinref part="R4" gate="1" pin="E"/>
+<wire x1="71.12" y1="22.86" x2="71.12" y2="25.4" width="0.1524" layer="91"/>
+<wire x1="63.5" y1="20.32" x2="63.5" y2="22.86" width="0.1524" layer="91"/>
+<wire x1="63.5" y1="22.86" x2="71.12" y2="22.86" width="0.1524" layer="91"/>
+<junction x="71.12" y="22.86"/>
+<label x="73.66" y="17.78" size="1.778" layer="95"/>
+<pinref part="JP1" gate="A" pin="2"/>
+<pinref part="P+3" gate="1" pin="+5V"/>
+</segment>
+<segment>
+<pinref part="JP1" gate="A" pin="19"/>
+<wire x1="83.82" y1="-25.4" x2="68.58" y2="-25.4" width="0.1524" layer="91"/>
+<pinref part="P+2" gate="1" pin="+5V"/>
+</segment>
+</net>
